File: schematic/power/power/power.kicad_pcb (KiCad board)
At the start: 2 copper layers, 99.1 x 68.6 mm, 23 parts, among them IC1 NCP5111PG, IC2 NCP5111PG, J1 1935161, J2 1935161, Q1 FQP17N40, Q2 FQP17N40, Q3 FQP17N40, Q4 FQP17N40, U1 74LS04

Commit message: add power ver 2
Routing:
- net VDD: track 42.1 -> 53.3 mm
- added copper zone on B.Cu, net GND
- added copper zone on F.Cu, net GND
Changed lines of the file:
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@@
     (thickness 1.6)
     (drawings 4)
-    (tracks 76)
+    (tracks 79)
     (zones 0)
     (modules 23)
@@
   )
   (setup
-    (last_trace_width 0.254)
+    (last_trace_width 0.508)
     (user_trace_width 0.254)
     (user_trace_width 0.508)
@@
     (pad 1 thru_hole rect (at -3.97 -3.81 90) (size 1.16 1.16) (drill 0.76) (layers *.Cu *.Mask F.SilkS)
       (net 1 +15V))
+    (model C:/Users/69134/Desktop/ECEN405_D_class_amp/schematic/lib/LIB_NCP5111PG/DIP794W56P254L959H533Q8N.kicad_mod
+      (at (xyz 0 0 0))
+      (scale (xyz 1 1 1))
+      (rotate (xyz 0 0 0))
+    )
+    (model C:/Users/69134/Desktop/ECEN405_D_class_amp/schematic/lib/LIB_NCP5111PG/NCP5111PG.mod
+      (at (xyz 0 0 0))
+      (scale (xyz 1 1 1))
+      (rotate (xyz 0 0 0))
+    )
   )
   (module TerminalBlock:TerminalBlock_Altech_AK300-2_P5.00mm (layer F.Cu)
@@
   (segment (start 151.13 107.95) (end 140.97 118.11) (width 0.508) (layer F.Cu) (net 5))
   (segment (start 153.67 107.95) (end 151.13 107.95) (width 0.508) (layer F.Cu) (net 5))
+  (segment (start 152.415999 106.695999) (end 153.67 107.95) (width 0.508) (layer F.Cu) (net 5))
+  (segment (start 152.415999 99.044001) (end 152.415999 106.695999) (width 0.508) (layer F.Cu) (net 5))
+  (segment (start 153.67 97.79) (end 152.415999 99.044001) (width 0.508) (layer F.Cu) (net 5))
   (segment (start 143.51 124.46) (end 140.97 127) (width 0.508) (layer F.Cu) (net 6))
   (segment (start 143.51 118.11) (end 143.51 124.46) (width 0.508) (layer F.Cu) (net 6))
@@
   (segment (start 102.87 123.03) (end 103.03 123.19) (width 0.508) (layer F.Cu) (net 7))
   (segment (start 102.87 115.57) (end 102.87 123.03) (width 0.508) (layer F.Cu) (net 7))
-  (segment (start 109.22 115.57) (end 111.76 113.03) (width 0.254) (layer F.Cu) (net 7))
-  (segment (start 102.87 115.57) (end 109.22 115.57) (width 0.254) (layer F.Cu) (net 7))
+  (segment (start 109.22 115.57) (end 111.76 113.03) (width 0.508) (layer F.Cu) (net 7))
+  (segment (start 102.87 115.57) (end 109.22 115.57) (width 0.508) (layer F.Cu) (net 7))
   (segment (start 86.36 100.33) (end 85.09 99.06) (width 0.254) (layer B.Cu) (net 8))
   (segment (start 95.09 100.33) (end 86.36 100.33) (width 0.254) (layer B.Cu) (net 8))
@@
   (segment (start 137.16 128.27) (end 138.43 127) (width 0.254) (layer F.Cu) (net 19))
   (segment (start 129.54 128.27) (end 137.16 128.27) (width 0.254) (layer F.Cu) (net 19))
+  (zone (net 2) (net_name GND) (layer F.Cu) (hatch edge 0.508)
+    (connect_pads (clearance 0.508))
+    (min_thickness 0.254)
+    (fill yes (arc_segments 32) (thermal_gap 0.508) (thermal_bridge_width 0.508))
+    (polygon
+      (pts
+        (xy 170.18 144.78) (xy 67.31 146.05) (xy 67.31 73.66) (xy 170.18 73.66)
+      )
+    )
+  )
+  (zone (net 2) (net_name GND) (layer B.Cu) (hatch edge 0.508)
+    (connect_pads (clearance 0.508))
+    (min_thickness 0.254)
+    (fill yes (arc_segments 32) (thermal_gap 0.508) (thermal_bridge_width 0.508))
+    (polygon
+      (pts
+        (xy 173.99 144.78) (xy 67.31 146.05) (xy 67.31 73.66) (xy 170.18 72.39)
+      )
+    )
+  )
 )
