File: schematic/power/power_ver_2.0/_autosave-power_ver_2.0.sch (KiCad schematic (older format))
At the start: 37 parts, among them J1 PWM INPUT, J2 Audio OUTPUT, J3 OUTPUT Power, J4 PWM_power, Q1 RFP12N10L, Q2 RFP12N10L, Q3 RFP12N10L, Q4 RFP12N10L, U1 HIP4082IP

Commit message: ver2 pcb layout
Parts:
- gave numbers to parts that had none: 4
Changed lines of the file:
@@
 $EndComp
 $Comp
-L Device:L L?
+L Device:L L2
 U 1 1 614D4A87
 P 8900 3750
-F 0 "L?" V 9090 3750 50  0000 C CNN
+F 0 "L2" V 9090 3750 50  0000 C CNN
 F 1 "2216-V-RC" V 8999 3750 50  0000 C CNN
 F 2 "Inductor_THT:L_Toroid_Vertical_L24.6mm_W15.5mm_P11.44mm_Pulse_KM-4" H 8900 3750 50  0001 C CNN
@@
 $EndComp
 $Comp
-L Device:C C?
+L Device:C C6
 U 1 1 614DAA49
 P 7450 4100
-F 0 "C?" H 7565 4146 50  0000 L CNN
+F 0 "C6" H 7565 4146 50  0000 L CNN
 F 1 "C324C106K3R5TA" H 7565 4055 50  0000 L CNN
 F 2 "Capacitor_THT:C_Radial_D4.0mm_H5.0mm_P1.50mm" H 7488 3950 50  0001 C CNN
@@
 $EndComp
 $Comp
-L Device:C C?
+L Device:C C9
 U 1 1 614DB54C
 P 8600 4100
-F 0 "C?" H 8715 4146 50  0000 L CNN
+F 0 "C9" H 8715 4146 50  0000 L CNN
 F 1 "C324C106K3R5TA" H 8715 4055 50  0000 L CNN
 F 2 "Capacitor_THT:C_Radial_D4.0mm_H5.0mm_P1.50mm" H 8638 3950 50  0001 C CNN
@@
 $EndComp
 $Comp
-L Device:C C?
+L Device:C C7
 U 1 1 614DC10B
 P 8000 3300
-F 0 "C?" V 7748 3300 50  0000 C CNN
+F 0 "C7" V 7748 3300 50  0000 C CNN
 F 1 "C324C106K3R5TA" V 7839 3300 50  0000 C CNN
 F 2 "Capacitor_THT:C_Radial_D4.0mm_H5.0mm_P1.50mm" H 8038 3150 50  0001 C CNN
