File: schematic/power/power_ver_2.0/_autosave-power_ver_2.0.sch (KiCad schematic (older format))
At the start: 47 parts, among them J1 PWM INPUT, J2 Audio OUTPUT, J3 Amp_Power, J4 Driver_power, Q1 IRF530A, Q2 IRF530A, Q3 IRF530A, Q4 IRF530A, U1 HIP4082IP

Commit message: labels
Parts:
- C10, C11, C2, C3: footprint Capacitor_THT:C_Radial_D4.0mm_H5.0mm_P1.50mm -> Capacitor_THT:C_Disc_D3.8mm_W2.6mm_P2.50mm
- gave numbers to parts that had none: 4
Changed lines of the file:
@@
 F 0 "C11" H 9565 2196 50  0000 L CNN
 F 1 "SR205C104MAATR1" H 9565 2105 50  0000 L CNN
-F 2 "Capacitor_THT:C_Radial_D4.0mm_H5.0mm_P1.50mm" H 9488 2000 50  0001 C CNN
+F 2 "Capacitor_THT:C_Disc_D3.8mm_W2.6mm_P2.50mm" H 9488 2000 50  0001 C CNN
 F 3 "~" H 9450 2150 50  0001 C CNN
 F 4 "0.1uF 50V 20%" H 9450 2150 50  0001 C CNN "Description"
@@
 F 0 "C2" H 2665 2996 50  0000 L CNN
 F 1 "C324C106K3R5TA" H 2500 3200 50  0000 L CNN
-F 2 "Capacitor_THT:C_Radial_D4.0mm_H5.0mm_P1.50mm" H 2588 2800 50  0001 C CNN
+F 2 "Capacitor_THT:C_Disc_D3.8mm_W2.6mm_P2.50mm" H 2588 2800 50  0001 C CNN
 F 3 "~" H 2550 2950 50  0001 C CNN
 	1    2550 2950
@@
 F 0 "C10" H 9115 2196 50  0000 L CNN
 F 1 "C324C106K3R5TA" H 9115 2105 50  0000 L CNN
-F 2 "Capacitor_THT:C_Radial_D4.0mm_H5.0mm_P1.50mm" H 9038 2000 50  0001 C CNN
+F 2 "Capacitor_THT:C_Disc_D3.8mm_W2.6mm_P2.50mm" H 9038 2000 50  0001 C CNN
 F 3 "~" H 9000 2150 50  0001 C CNN
 F 4 "10uF 25V 10%" H 9000 2150 50  0001 C CNN "Description"
@@
 F 0 "C3" H 3115 2996 50  0000 L CNN
 F 1 "SR205C104MAATR1" H 3050 2850 50  0000 L CNN
-F 2 "Capacitor_THT:C_Radial_D4.0mm_H5.0mm_P1.50mm" H 3038 2800 50  0001 C CNN
+F 2 "Capacitor_THT:C_Disc_D3.8mm_W2.6mm_P2.50mm" H 3038 2800 50  0001 C CNN
 F 3 "~" H 3000 2950 50  0001 C CNN
 F 4 "0.1uF 50V 20%" H 3000 2950 50  0001 C CNN "Description"
@@
 	1    0    0    -1
 $EndComp
-Connection ~ 10300 4250
 Connection ~ 6150 2750
 Connection ~ 6200 4250
-Connection ~ 5400 3950
-Wire Wire Line
-	5400 3950 5700 3950
-Wire Wire Line
-	4350 3950 5400 3950
 Connection ~ 5900 4450
 Wire Wire Line
@@
 Connection ~ 10050 2850
 $Comp
-L Mechanical:MountingHole H?
+L Mechanical:MountingHole H1
 U 1 1 61545B32
 P 1150 7000
-F 0 "H?" H 1250 7046 50  0000 L CNN
+F 0 "H1" H 1250 7046 50  0000 L CNN
 F 1 "MountingHole" H 1250 6955 50  0000 L CNN
 F 2 "MountingHole:MountingHole_4.3mm_M4" H 1150 7000 50  0001 C CNN
@@
 $EndComp
 $Comp
-L Mechanical:MountingHole H?
+L Mechanical:MountingHole H2
 U 1 1 61546C2A
 P 2000 7000
-F 0 "H?" H 2100 7046 50  0000 L CNN
+F 0 "H2" H 2100 7046 50  0000 L CNN
 F 1 "MountingHole" H 2100 6955 50  0000 L CNN
 F 2 "MountingHole:MountingHole_4.3mm_M4" H 2000 7000 50  0001 C CNN
@@
 $EndComp
 $Comp
-L Mechanical:MountingHole H?
+L Mechanical:MountingHole H3
 U 1 1 61547715
 P 2800 7000
-F 0 "H?" H 2900 7046 50  0000 L CNN
+F 0 "H3" H 2900 7046 50  0000 L CNN
 F 1 "MountingHole" H 2900 6955 50  0000 L CNN
 F 2 "MountingHole:MountingHole_4.3mm_M4" H 2800 7000 50  0001 C CNN
@@
 $EndComp
 $Comp
-L Mechanical:MountingHole H?
+L Mechanical:MountingHole H4
 U 1 1 61547A96
 P 3600 7000
-F 0 "H?" H 3700 7046 50  0000 L CNN
+F 0 "H4" H 3700 7046 50  0000 L CNN
 F 1 "MountingHole" H 3700 6955 50  0000 L CNN
 F 2 "MountingHole:MountingHole_4.3mm_M4" H 3600 7000 50  0001 C CNN
@@
 	1    0    0    -1
 $EndComp
+Wire Wire Line
+	4350 3950 5700 3950
 $EndSCHEMATC
