File: schematic/power/power_ver_2.0/power_ver_2.0.sch (KiCad schematic (older format))
At the start: 37 parts, among them J1 PWM INPUT, J2 Audio OUTPUT, J3 OUTPUT Power, J4 PWM_power, Q1 RFP12N10L, Q2 RFP12N10L, Q3 RFP12N10L, Q4 RFP12N10L, U1 HIP4082IP

Commit message: finish pcb trace layout
Parts:
- removed Q1, Q2, Q3, Q4: RFP12N10L, digikey-footprints:TO-220-3, symbol dk_Transistors-FETs-MOSFETs-Single:FQP30N06L
- added Q1, Q2, Q3, Q4: IRF530A, digikey-footprints:TO-220-3, symbol dk_Transistors-FETs-MOSFETs-Single:IRF540NPBF
- added R10, R11: 470, Resistor_THT:R_Axial_DIN0207_L6.3mm_D2.5mm_P10.16mm_Horizontal, symbol Device:R
- C6, C7, C9: renamed from C?; footprint Capacitor_THT:C_Radial_D4.0mm_H5.0mm_P1.50mm -> Capacitor_THT:C_Radial_D5.0mm_H11.0mm_P2.00mm
- J3: value OUTPUT Power -> Amp_Power
- J4: value PWM_power -> Driver_power
- R2, R3, R8, R9: value R -> 100
- R4, R5, R6, R7: value R -> 10k
- gave numbers to parts that had none: 1
Connections:
- net labels added: +10V, AHO, ALO, A_HI, A_LO, BHO, BLO, B_HI, B_LO
- net labels removed: +5V
- wire segments 116 -> 123
Other:
- moved on the sheet: J3

Commit message: add mounting hole, test point
Parts:
- added H? (x4): MountingHole, MountingHole:MountingHole_4.3mm_M4, symbol Mechanical:MountingHole
- added TP1, TP2, TP3, TP4: TestPoint, TestPoint:TestPoint_THTPad_D2.0mm_Drill1.0mm, symbol Connector:TestPoint
- C6, C7, C9: footprint Capacitor_THT:C_Radial_D5.0mm_H11.0mm_P2.00mm -> Capacitor_THT:C_Radial_D10.0mm_H12.5mm_P5.00mm
Connections:
- net at D3.2 (A), Q1.1 (G), R2.1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: now also TP1.1
- net at D4.2 (A), Q2.1 (G), R3.1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: now also TP2.1
- net at D6.2 (A), Q3.1 (G), R7.2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: now also TP4.1
- net at D5.2 (A), Q4.1 (G), R6.2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: now also TP3.1
Changed lines of the file:
@@
 	4350 4050 4350 3950
-Wire Wire Line
-	4350 3950 5700 3950
 Wire Wire Line
 	5700 3950 5700 3000
@@
 	4100 5050 10550 5050
 Wire Wire Line
-	10550 5050 10550 3050
-Wire Wire Line
 	10550 3050 10350 3050
 Wire Wire Line
@@
 Wire Wire Line
 	5850 3750 6500 3750
-Wire Wire Line
-	4300 4450 5900 4450
 $Comp
 L Diode:1N4148 D4
@@
 Wire Wire Line
 	5900 4250 5900 4450
-Connection ~ 5900 4450
 Wire Wire Line
 	6200 4250 6200 4450
@@
 F 0 "C6" H 7565 4146 50  0000 L CNN
 F 1 "C324C106K3R5TA" H 7565 4055 50  0000 L CNN
-F 2 "Capacitor_THT:C_Radial_D5.0mm_H11.0mm_P2.00mm" H 7488 3950 50  0001 C CNN
+F 2 "Capacitor_THT:C_Radial_D10.0mm_H12.5mm_P5.00mm" H 7488 3950 50  0001 C CNN
 F 3 "~" H 7450 4100 50  0001 C CNN
 F 4 "10uF 25V 10%" H 7450 4100 50  0001 C CNN "Description"
@@
 F 0 "C9" H 8715 4146 50  0000 L CNN
 F 1 "C324C106K3R5TA" H 8715 4055 50  0000 L CNN
-F 2 "Capacitor_THT:C_Radial_D5.0mm_H11.0mm_P2.00mm" H 8638 3950 50  0001 C CNN
+F 2 "Capacitor_THT:C_Radial_D10.0mm_H12.5mm_P5.00mm" H 8638 3950 50  0001 C CNN
 F 3 "~" H 8600 4100 50  0001 C CNN
 F 4 "10uF 25V 10%" H 8600 4100 50  0001 C CNN "Description"
@@
 F 0 "C7" V 7748 3300 50  0000 C CNN
 F 1 "C324C106K3R5TA" V 7839 3300 50  0000 C CNN
-F 2 "Capacitor_THT:C_Radial_D5.0mm_H11.0mm_P2.00mm" H 8038 3150 50  0001 C CNN
+F 2 "Capacitor_THT:C_Radial_D10.0mm_H12.5mm_P5.00mm" H 8038 3150 50  0001 C CNN
 F 3 "~" H 8000 3300 50  0001 C CNN
 F 4 "10uF 25V 10%" H 8000 3300 50  0001 C CNN "Description"
@@
 Wire Wire Line
 	3750 1500 4300 1500
+$Comp
+L Connector:TestPoint TP1
+U 1 1 61480284
+P 6150 2750
+F 0 "TP1" H 6208 2868 50  0000 L CNN
+F 1 "TestPoint" H 6208 2777 50  0000 L CNN
+F 2 "TestPoint:TestPoint_THTPad_D2.0mm_Drill1.0mm" H 6350 2750 50  0001 C CNN
+F 3 "~" H 6350 2750 50  0001 C CNN
+	1    6150 2750
+	1    0    0    -1
+$EndComp
+$Comp
+L Connector:TestPoint TP2
+U 1 1 6148304D
+P 6200 4250
+F 0 "TP2" H 6258 4368 50  0000 L CNN
+F 1 "TestPoint" H 6258 4277 50  0000 L CNN
+F 2 "TestPoint:TestPoint_THTPad_D2.0mm_Drill1.0mm" H 6400 4250 50  0001 C CNN
+F 3 "~" H 6400 4250 50  0001 C CNN
+	1    6200 4250
+	1    0    0    -1
+$EndComp
+$Comp
+L Connector:TestPoint TP3
+U 1 1 61492C2E
+P 9950 4250
+F 0 "TP3" H 10008 4368 50  0000 L CNN
+F 1 "TestPoint" H 10008 4277 50  0000 L CNN
+F 2 "TestPoint:TestPoint_THTPad_D2.0mm_Drill1.0mm" H 10150 4250 50  0001 C CNN
+F 3 "~" H 10150 4250 50  0001 C CNN
+	1    9950 4250
+	1    0    0    -1
+$EndComp
+Wire Wire Line
+	10550 5050 10550 3050
+$Comp
+L Connector:TestPoint TP4
+U 1 1 6148E53F
+P 10050 2850
+F 0 "TP4" H 10108 2968 50  0000 L CNN
+F 1 "TestPoint" H 10108 2877 50  0000 L CNN
+F 2 "TestPoint:TestPoint_THTPad_D2.0mm_Drill1.0mm" H 10250 2850 50  0001 C CNN
+F 3 "~" H 10250 2850 50  0001 C CNN
+	1    10050 2850
+	1    0    0    -1
+$EndComp
+Connection ~ 10300 4250
+Connection ~ 6150 2750
+Connection ~ 6200 4250
+Connection ~ 5400 3950
+Wire Wire Line
+	5400 3950 5700 3950
+Wire Wire Line
+	4350 3950 5400 3950
+Connection ~ 5900 4450
+Wire Wire Line
+	4300 4450 5900 4450
+Connection ~ 9950 4250
+Connection ~ 10050 2850
+$Comp
+L Mechanical:MountingHole H?
+U 1 1 61545B32
+P 1150 7000
+F 0 "H?" H 1250 7046 50  0000 L CNN
+F 1 "MountingHole" H 1250 6955 50  0000 L CNN
+F 2 "MountingHole:MountingHole_4.3mm_M4" H 1150 7000 50  0001 C CNN
+F 3 "~" H 1150 7000 50  0001 C CNN
+	1    1150 7000
+	1    0    0    -1
+$EndComp
+$Comp
+L Mechanical:MountingHole H?
+U 1 1 61546C2A
+P 2000 7000
+F 0 "H?" H 2100 7046 50  0000 L CNN
+F 1 "MountingHole" H 2100 6955 50  0000 L CNN
+F 2 "MountingHole:MountingHole_4.3mm_M4" H 2000 7000 50  0001 C CNN
+F 3 "~" H 2000 7000 50  0001 C CNN
+	1    2000 7000
+	1    0    0    -1
+$EndComp
+$Comp
+L Mechanical:MountingHole H?
+U 1 1 61547715
+P 2800 7000
+F 0 "H?" H 2900 7046 50  0000 L CNN
+F 1 "MountingHole" H 2900 6955 50  0000 L CNN
+F 2 "MountingHole:MountingHole_4.3mm_M4" H 2800 7000 50  0001 C CNN
+F 3 "~" H 2800 7000 50  0001 C CNN
+	1    2800 7000
+	1    0    0    -1
+$EndComp
+$Comp
+L Mechanical:MountingHole H?
+U 1 1 61547A96
+P 3600 7000
+F 0 "H?" H 3700 7046 50  0000 L CNN
+F 1 "MountingHole" H 3700 6955 50  0000 L CNN
+F 2 "MountingHole:MountingHole_4.3mm_M4" H 3600 7000 50  0001 C CNN
+F 3 "~" H 3600 7000 50  0001 C CNN
+	1    3600 7000
+	1    0    0    -1
+$EndComp
 $EndSCHEMATC

Commit message: labels
Parts:
- C10, C11, C2, C3: footprint Capacitor_THT:C_Radial_D4.0mm_H5.0mm_P1.50mm -> Capacitor_THT:C_Disc_D3.8mm_W2.6mm_P2.50mm
- gave numbers to parts that had none: 4
Changed lines of the file:
@@
 F 0 "C11" H 9565 2196 50  0000 L CNN
 F 1 "SR205C104MAATR1" H 9565 2105 50  0000 L CNN
-F 2 "Capacitor_THT:C_Radial_D4.0mm_H5.0mm_P1.50mm" H 9488 2000 50  0001 C CNN
+F 2 "Capacitor_THT:C_Disc_D3.8mm_W2.6mm_P2.50mm" H 9488 2000 50  0001 C CNN
 F 3 "~" H 9450 2150 50  0001 C CNN
 F 4 "0.1uF 50V 20%" H 9450 2150 50  0001 C CNN "Description"
@@
 F 0 "C2" H 2665 2996 50  0000 L CNN
 F 1 "C324C106K3R5TA" H 2500 3200 50  0000 L CNN
-F 2 "Capacitor_THT:C_Radial_D4.0mm_H5.0mm_P1.50mm" H 2588 2800 50  0001 C CNN
+F 2 "Capacitor_THT:C_Disc_D3.8mm_W2.6mm_P2.50mm" H 2588 2800 50  0001 C CNN
 F 3 "~" H 2550 2950 50  0001 C CNN
 	1    2550 2950
@@
 F 0 "C10" H 9115 2196 50  0000 L CNN
 F 1 "C324C106K3R5TA" H 9115 2105 50  0000 L CNN
-F 2 "Capacitor_THT:C_Radial_D4.0mm_H5.0mm_P1.50mm" H 9038 2000 50  0001 C CNN
+F 2 "Capacitor_THT:C_Disc_D3.8mm_W2.6mm_P2.50mm" H 9038 2000 50  0001 C CNN
 F 3 "~" H 9000 2150 50  0001 C CNN
 F 4 "10uF 25V 10%" H 9000 2150 50  0001 C CNN "Description"
@@
 F 0 "C3" H 3115 2996 50  0000 L CNN
 F 1 "SR205C104MAATR1" H 3050 2850 50  0000 L CNN
-F 2 "Capacitor_THT:C_Radial_D4.0mm_H5.0mm_P1.50mm" H 3038 2800 50  0001 C CNN
+F 2 "Capacitor_THT:C_Disc_D3.8mm_W2.6mm_P2.50mm" H 3038 2800 50  0001 C CNN
 F 3 "~" H 3000 2950 50  0001 C CNN
 F 4 "0.1uF 50V 20%" H 3000 2950 50  0001 C CNN "Description"
@@
 Connection ~ 10050 2850
 $Comp
-L Mechanical:MountingHole H?
+L Mechanical:MountingHole H1
 U 1 1 61545B32
 P 1150 7000
-F 0 "H?" H 1250 7046 50  0000 L CNN
+F 0 "H1" H 1250 7046 50  0000 L CNN
 F 1 "MountingHole" H 1250 6955 50  0000 L CNN
 F 2 "MountingHole:MountingHole_4.3mm_M4" H 1150 7000 50  0001 C CNN
@@
 $EndComp
 $Comp
-L Mechanical:MountingHole H?
+L Mechanical:MountingHole H2
 U 1 1 61546C2A
 P 2000 7000
-F 0 "H?" H 2100 7046 50  0000 L CNN
+F 0 "H2" H 2100 7046 50  0000 L CNN
 F 1 "MountingHole" H 2100 6955 50  0000 L CNN
 F 2 "MountingHole:MountingHole_4.3mm_M4" H 2000 7000 50  0001 C CNN
@@
 $EndComp
 $Comp
-L Mechanical:MountingHole H?
+L Mechanical:MountingHole H3
 U 1 1 61547715
 P 2800 7000
-F 0 "H?" H 2900 7046 50  0000 L CNN
+F 0 "H3" H 2900 7046 50  0000 L CNN
 F 1 "MountingHole" H 2900 6955 50  0000 L CNN
 F 2 "MountingHole:MountingHole_4.3mm_M4" H 2800 7000 50  0001 C CNN
@@
 $EndComp
 $Comp
-L Mechanical:MountingHole H?
+L Mechanical:MountingHole H4
 U 1 1 61547A96
 P 3600 7000
-F 0 "H?" H 3700 7046 50  0000 L CNN
+F 0 "H4" H 3700 7046 50  0000 L CNN
 F 1 "MountingHole" H 3700 6955 50  0000 L CNN
 F 2 "MountingHole:MountingHole_4.3mm_M4" H 3600 7000 50  0001 C CNN

Commit message: add BOM
Parts:
- C11, C3: value SR205C104MAATR1 -> K104Z15Y5VE5TL2; Description 0.1uF 50V 20% -> 0.1uF 25V -20%,+80%
- C2: Description (none) -> 10uF 25V 10%
- C4, C5: value ECE-A1HN100U -> ECA-1EM100B; footprint Capacitor_THT:CP_Radial_D6.3mm_P2.50mm -> Capacitor_THT:CP_Radial_Tantal_D5.0mm_P5.00mm; Description 10uF 50V 20% -> 10uF 25V 20%
- C6, C7, C9: value C324C106K3R5TA -> uF; Description 10uF 25V 10% -> (none)
- D1, D2, D3, D4, D5, D6: Description (none) -> 100V 200mA; Digi-Key_PN (none) -> 1N4148FS-ND
- J1, J2, J3, J4: Digi-Key_PN (none) -> 277-1667-ND
- Q1, Q2, Q3, Q4: Category Discrete Semiconductor Products -> (none); Family Transistors - FETs, MOSFETs - Single -> (none); Status Active -> (none)
- R1: value 1K -> MFP-25BRD52-1K; Description (none) -> 1k ohm 1% 1/4w
- R10, R11: value 470 -> CFR-25JB-52-470R; Description (none) -> 470 ohm 5% 1/4W
- R2, R3, R8, R9: value 100 -> CFR-25JR-52-100R; Description (none) -> 100 ohm 5% 1/4W
- R4, R5, R6, R7: value 10k -> CFR50SJT-52-10K; Description (none) -> 10k ohm 5% 1/4W
- U1: Description (none) -> Full bridge gate driver
Connections:
- net A_HI: no longer names the net of C4.1, L2.2, Q3.3 (S), Q4.2 (D), R7.1, U1.11 (AHS)
- net B_HI: no longer names the net of C5.2, L1.1, Q1.3 (S), Q2.2 (D), R4.1, U1.15 (BHS)
Other:
- moved on the sheet: TP2, TP3, TP4
