File: schematic/joint_pcb/low_pass_filter_stage.sch (KiCad schematic (older format))
At the start: 5 parts

Commit message: Fixed PCB
Parts:
- C24: symbol C4AQLBW6130A3NK:C4AQLBW6130A3NK -> joint_pcb-rescue:C4AQLBW6130A3NK-C4AQLBW6130A3NK
Changed lines of the file:
@@
 $EndComp
 $Comp
-L C4AQLBW6130A3NK:C4AQLBW6130A3NK C24
+L joint_pcb-rescue:C4AQLBW6130A3NK-C4AQLBW6130A3NK C24
 U 1 1 61363422
 P 5300 3200
