File: schematic/joint_pcb/input_stage.sch (KiCad schematic (older format))
At the start: 39 parts, among them IC1 ADA4891-2ARMZ-R7, IC2 LM361N_NOPB, J1 Screw_Terminal_01x04, U1 LM7805_TO220, U2 LM324

Commit message: Fixed PCB
Parts:
- IC1: symbol ADA4891-2ARMZ-R7:ADA4891-2ARMZ-R7 -> joint_pcb-rescue:ADA4891-2ARMZ-R7-ADA4891-2ARMZ-R7
- IC2: symbol LM361:LM361N_NOPB -> joint_pcb-rescue:LM361N_NOPB-LM361
Connections:
- net +10V renamed +15V
Changed lines of the file:
@@
 $EndComp
 $Comp
-L ADA4891-2ARMZ-R7:ADA4891-2ARMZ-R7 IC1
+L joint_pcb-rescue:ADA4891-2ARMZ-R7-ADA4891-2ARMZ-R7 IC1
 U 1 1 6112424A
 P 3600 4950
+AR Path="/6112424A" Ref="IC1"  Part="1"
+AR Path="/6131B79C/6112424A" Ref="IC1"  Part="1"
 F 0 "IC1" H 4200 5215 50  0000 C CNN
 F 1 "ADA4891-2ARMZ-R7" H 4200 5124 50  0000 C CNN
@@
 $EndComp
 $Comp
-L LM361:LM361N_NOPB IC2
+L joint_pcb-rescue:LM361N_NOPB-LM361 IC2
 U 1 1 611DBEC5
 P 6200 4750
@@
 Text Notes 1150 4200 0    118  ~ 0
 Input
-Text GLabel 850  4650 0    50   Input ~ 0
+Text GLabel 800  4650 0    50   Input ~ 0
 Vcc
 Text GLabel 2200 2800 3    50   Input ~ 0
@@
 Wire Wire Line
 	7700 5250 8250 5250
-$Comp
-L power:+10V #PWR01
-U 1 1 613AC109
-P 900 4300
-F 0 "#PWR01" H 900 4150 50  0001 C CNN
-F 1 "+10V" H 915 4473 50  0000 C CNN
-F 2 "" H 900 4300 50  0001 C CNN
-F 3 "" H 900 4300 50  0001 C CNN
-	1    900  4300
-	1    0    0    -1
-$EndComp
-Wire Wire Line
-	850  4650 900  4650
-Wire Wire Line
-	900  4300 900  4650
-Connection ~ 900  4650
-Wire Wire Line
-	900  4650 1150 4650
+Wire Wire Line
+	800  4650 850  4650
+Wire Wire Line
+	850  4300 850  4650
+Connection ~ 850  4650
+$Comp
+L power:+15V #PWR?
+U 1 1 613910BD
+P 850 4300
+F 0 "#PWR?" H 850 4150 50  0001 C CNN
+F 1 "+15V" H 865 4473 50  0000 C CNN
+F 2 "" H 850 4300 50  0001 C CNN
+F 3 "" H 850 4300 50  0001 C CNN
+	1    850  4300
+	1    0    0    -1
+$EndComp
+Wire Wire Line
+	850  4650 1150 4650
 $EndSCHEMATC
