File: schematic/joint_pcb/joint_pcb.sch (KiCad schematic (older format))
At the start: 0 parts

Commit message: finish layout for PCB
Changed lines of the file:
@@
 $Descr A4 11693 8268
 encoding utf-8
-Sheet 1 4
+Sheet 1 3
 Title ""
 Date ""
@@
 F5 "OUT-" O R 7000 4100 50
 $EndSheet
-$Sheet
-S 7800 3050 2100 1600
-U 6133C589
-F0 "Low-pass filter stage" 50
-F1 "low_pass_filter_stage.sch" 50
-F2 "IN+" I L 7800 3550 50
-F3 "IN-" I L 7800 4100 50
-$EndSheet
-Wire Wire Line
-	7000 3550 7800 3550
-Wire Wire Line
-	7000 4100 7800 4100
 Wire Wire Line
 	4000 3450 4850 3450
