File: schematic/joint_pcb_ver2/input_stage.sch (KiCad schematic (older format))
At the start: 39 parts, among them IC1 ADA4891-2ARMZ-R7, IC2 LM361N_NOPB, J1 Screw_Terminal_01x04, U1 LM7805_TO220, U2 LM324

Commit message: connect up 10V
Connections:
- net +15V renamed +10V
Changed lines of the file:
@@
 $Descr A4 11693 8268
 encoding utf-8
-Sheet 2 4
+Sheet 2 3
 Title ""
 Date ""
@@
 	850  4300 850  4650
 Connection ~ 850  4650
-$Comp
-L power:+15V #PWR?
-U 1 1 613910BD
+Wire Wire Line
+	850  4650 1150 4650
+$Comp
+L power:+10V #PWR023
+U 1 1 613F4FD9
 P 850 4300
-F 0 "#PWR?" H 850 4150 50  0001 C CNN
-F 1 "+15V" H 865 4473 50  0000 C CNN
+F 0 "#PWR023" H 850 4150 50  0001 C CNN
+F 1 "+10V" H 865 4473 50  0000 C CNN
 F 2 "" H 850 4300 50  0001 C CNN
 F 3 "" H 850 4300 50  0001 C CNN
@@
 	1    0    0    -1
 $EndComp
-Wire Wire Line
-	850  4650 1150 4650
 $EndSCHEMATC
