File: schematic/power/power_ver_3.0/power_ver_3.0.kicad_pcb (KiCad board)
At the start: 2 copper layers, 29 parts, among them J1 Power_PWM_output, J2 Amp_power, Q1 IRF510PBF, Q2 IRF510PBF, Q3 IRF510PBF, Q4 IRF510PBF, U1 HIP4081AIPZ

Commit message: power 3.0 pcb layout
Parts:
- moved R1 53.2 mm to (60.7, 66.3), turned to 270 degrees
- moved C8 49.8 mm to (103.4, 48.0), turned to 90 degrees
- moved R2 49.2 mm to (65.8, 68.8), turned to 270 degrees
- moved C9 48.8 mm to (111.0, 48.0), turned to 90 degrees
- moved C7 48.6 mm to (123.2, 47.0)
- moved J1 42.9 mm to (146.3, 76.2)
- moved R4 42.7 mm to (70.9, 84.1), turned to 90 degrees
- moved Q4 42.0 mm to (138.4, 77.0)
- moved Q3 41.5 mm to (138.4, 63.2)
- moved C6 39.3 mm to (86.9, 48.5)
- moved U1 37.6 mm to (85.6, 56.1)
- moved Q2 37.5 mm to (123.2, 77.0)
- moved C3 37.0 mm to (73.2, 57.4)
- moved Q1 36.9 mm to (123.2, 63.2)
- moved D4 36.5 mm to (103.4, 65.8)
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Connections:
- net ALS renamed GND

Commit message: finish layout for PCB
Routing:
- net BHS: track 0.00 -> 99.2 mm
- net AHS: track 0.00 -> 75.9 mm
- net +10V: track 0.00 -> 72.7 mm
- net +15V: track 0.00 -> 64.9 mm
- net Net-(D6-Pad2): track 0.00 -> 46.4 mm
- net Net-(D5-Pad2): track 0.00 -> 34.0 mm
- net Net-(R1-Pad1): track 0.00 -> 24.9 mm
- net Net-(D4-Pad2): track 0.00 -> 22.9 mm
- net Net-(D3-Pad2): track 0.00 -> 20.6 mm
- net Net-(R2-Pad1): track 0.00 -> 19.8 mm
- net Net-(R3-Pad2): track 0.00 -> 14.7 mm
- net Net-(C4-Pad1): track 0.00 -> 14.6 mm
- net ALO: track 0.00 -> 14.3 mm
- net AHO: track 0.00 -> 14.3 mm
- net Net-(C6-Pad1): track 0.00 -> 14.3 mm
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
Commit message: connect up 10V
Connections:
- net +10V renamed Vcc
